File: PokeyMax4/Decoupling.kicad_sch (KiCad schematic)
At the start: 5 parts

Commit message: Update the v4 board
Parts:
- C1, C11, C2, C5, C6: JLCPCB Part # C126523 -> (none); LCSC Part # (none) -> C141382

Commit message: Updates for JLCPCB fabrication and parts library
Parts:
- C1, C11, C2, C5, C6: LCSC Part # C141382 -> C1525
Changed lines of the file:
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@@
 	(global_label "3V3"
 		(shape bidirectional)
-		(at 157.48 87.63 0)
+		(at 157.48 81.28 0)
 		(fields_autoplaced yes)
 		(effects
@@
 		)
 		(property "Intersheetrefs" "${INTERSHEET_REFS}"
-			(at 164.9316 87.63 0)
+			(at 164.9316 81.28 0)
 			(effects
 				(font
@@
 	(global_label "2V5"
 		(shape bidirectional)
-		(at 116.84 86.36 90)
+		(at 116.84 81.28 90)
 		(fields_autoplaced yes)
 		(effects
@@
 		)
 		(property "Intersheetrefs" "${INTERSHEET_REFS}"
-			(at 116.84 78.9084 90)
+			(at 116.84 73.8284 90)
 			(effects
 				(font
@@
 	(global_label "5V0"
 		(shape bidirectional)
-		(at 172.72 88.9 0)
+		(at 172.72 86.36 0)
 		(fields_autoplaced yes)
 		(effects
@@
 		)
 		(property "Intersheetrefs" "${INTERSHEET_REFS}"
-			(at 180.1716 88.9 0)
+			(at 180.1716 86.36 0)
 			(effects
 				(font
@@
 			)
 		)
-		(property "LCSC Part #" "C141382"
+		(property "LCSC Part #" " C1525"
+			(at 172.72 96.52 0)
+			(effects
+				(font
+					(size 1.27 1.27)
+				)
+				(hide yes)
+			)
+		)
+		(property "JLCPCB Rotation Offset" ""
 			(at 172.72 96.52 0)
 			(effects
@@
 			)
 		)
-		(property "LCSC Part #" "C141382"
+		(property "LCSC Part #" " C1525"
+			(at 142.24 96.52 0)
+			(effects
+				(font
+					(size 1.27 1.27)
+				)
+				(hide yes)
+			)
+		)
+		(property "JLCPCB Rotation Offset" ""
 			(at 142.24 96.52 0)
 			(effects
@@
 			)
 		)
-		(property "LCSC Part #" "C141382"
+		(property "LCSC Part #" " C1525"
+			(at 157.48 96.52 0)
+			(effects
+				(font
+					(size 1.27 1.27)
+				)
+				(hide yes)
+			)
+		)
+		(property "JLCPCB Rotation Offset" ""
 			(at 157.48 96.52 0)
 			(effects
@@
 			)
 		)
-		(property "LCSC Part #" "C141382"
+		(property "LCSC Part #" " C1525"
+			(at 116.84 96.52 0)
+			(effects
+				(font
+					(size 1.27 1.27)
+				)
+				(hide yes)
+			)
+		)
+		(property "JLCPCB Rotation Offset" ""
 			(at 116.84 96.52 0)
 			(effects
@@
 			)
 		)
-		(property "LCSC Part #" "C141382"
+		(property "LCSC Part #" " C1525"
 			(at 132.08 96.52 0)
 			(effects
+				(font
+					(size 1.27 1.27)
+				)
+				(hide yes)
+			)
+		)
+		(property "JLCPCB Rotation Offset" ""
+			(at 132.08 96.52 0)
+			(effects

Commit message: Update BOM from 0402 to 0603 where relevant
Parts:
- C1, C11, C2, C5, C6: LCSC Part # C1525 -> C88219
Changed lines of the file:
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@@
 			)
 		)
-		(property "LCSC Part #" " C1525"
+		(property "LCSC Part #" "C88219"
 			(at 172.72 96.52 0)
 			(effects
@@
 			)
 		)
-		(property "LCSC Part #" " C1525"
+		(property "LCSC Part #" "C88219"
 			(at 142.24 96.52 0)
 			(effects
@@
 			)
 		)
-		(property "LCSC Part #" " C1525"
+		(property "LCSC Part #" "C88219"
 			(at 157.48 96.52 0)
 			(effects
@@
 			)
 		)
-		(property "LCSC Part #" " C1525"
+		(property "LCSC Part #" "C88219"
 			(at 116.84 96.52 0)
 			(effects
@@
 			)
 		)
-		(property "LCSC Part #" " C1525"
+		(property "LCSC Part #" "C88219"
 			(at 132.08 96.52 0)
 			(effects
