File: PokeyMax4/FPGA.kicad_sch (KiCad schematic)
At the start: 11 parts, among them U3 MAX10, X1 ASE

Commit message: Update the v4 board
Parts:
- C10: JLCPCB Part # C323592 -> (none); LCSC Part # (none) -> C15195
- FB1: JLCPCB Part # C710330 -> (none); LCSC Part # (none) -> C710330
- JTAG0: LCSC Part # (none) -> C2913924
- R1, R2, R4, R5: JLCPCB Part # C2654118 -> (none); LCSC Part # (none) -> C25744
- R3: JLCPCB Part # C11702 -> (none); LCSC Part # (none) -> C11702
- REG2: JLCPCB Part # C622555 -> (none); LCSC Part # (none) -> C622559
- U3: JLCPCB Part # C131386 -> (none); LCSC Part # (none) -> C1521934
- X1: JLCPCB Part # C1179056 -> (none); LCSC Part # (none) -> C1179056

Commit message: Updates for JLCPCB fabrication and parts library
Parts:
- JTAG0: LCSC Part # C2913924 -> (none); now left out of the parts list
- REG2: JLCPCB Rotation Offset (none) -> 270
- U3: LCSC Part # C1521934 -> C1521935
- X1: LCSC Part # C1179056 -> C7431354
Changed lines of the file:
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@@
 	(global_label "GND"
 		(shape bidirectional)
-		(at 57.15 154.94 0)
-		(fields_autoplaced yes)
-		(effects
-			(font
-				(size 1.2446 1.2446)
-			)
-			(justify left)
-		)
-		(property "Intersheetrefs" "${INTERSHEET_REFS}"
-			(at 64.9573 154.94 0)
+		(at 53.34 154.94 180)
+		(fields_autoplaced yes)
+		(effects
+			(font
+				(size 1.2446 1.2446)
+			)
+			(justify right)
+		)
+		(property "Intersheetrefs" "${INTERSHEET_REFS}"
+			(at 61.1473 154.94 0)
 			(effects
 				(font
@@
 	(global_label "GND"
 		(shape bidirectional)
-		(at 121.92 121.92 0)
-		(fields_autoplaced yes)
-		(effects
-			(font
-				(size 1.2446 1.2446)
-			)
-			(justify left)
-		)
-		(property "Intersheetrefs" "${INTERSHEET_REFS}"
-			(at 129.7273 121.92 0)
+		(at 111.76 121.92 180)
+		(fields_autoplaced yes)
+		(effects
+			(font
+				(size 1.2446 1.2446)
+			)
+			(justify right)
+		)
+		(property "Intersheetrefs" "${INTERSHEET_REFS}"
+			(at 119.5673 121.92 0)
 			(effects
 				(font
@@
 	(global_label "3V3"
 		(shape bidirectional)
-		(at 101.6 154.94 0)
-		(fields_autoplaced yes)
-		(effects
-			(font
-				(size 1.2446 1.2446)
-			)
-			(justify left)
-		)
-		(property "Intersheetrefs" "${INTERSHEET_REFS}"
-			(at 109.0516 154.94 0)
+		(at 109.22 154.94 0)
+		(fields_autoplaced yes)
+		(effects
+			(font
+				(size 1.2446 1.2446)
+			)
+			(justify left)
+		)
+		(property "Intersheetrefs" "${INTERSHEET_REFS}"
+			(at 116.6716 154.94 0)
 			(effects
 				(font
@@
 	(global_label "GND"
 		(shape bidirectional)
-		(at 101.6 152.4 0)
-		(fields_autoplaced yes)
-		(effects
-			(font
-				(size 1.2446 1.2446)
-			)
-			(justify left)
-		)
-		(property "Intersheetrefs" "${INTERSHEET_REFS}"
-			(at 109.4073 152.4 0)
+		(at 106.68 152.4 0)
+		(fields_autoplaced yes)
+		(effects
+			(font
+				(size 1.2446 1.2446)
+			)
+			(justify left)
+		)
+		(property "Intersheetrefs" "${INTERSHEET_REFS}"
+			(at 114.4873 152.4 0)
 			(effects
 				(font
@@
 	(global_label "2V5"
 		(shape bidirectional)
-		(at 58.42 152.4 0)
-		(fields_autoplaced yes)
-		(effects
-			(font
-				(size 1.2446 1.2446)
-			)
-			(justify left)
+		(at 58.42 152.4 180)
+		(fields_autoplaced yes)
+		(effects
+			(font
+				(size 1.2446 1.2446)
+			)
+			(justify right)
 		)
 		(property "Intersheetrefs" "${INTERSHEET_REFS}"
@@
 			)
 		)
+		(property "JLCPCB Rotation Offset" ""
+			(at 127 109.22 0)
+			(effects
+				(font
+					(size 1.27 1.27)
+				)
+				(hide yes)
+			)
+		)
 		(pin "1"
 		)
@@
 			)
 		)
+		(property "JLCPCB Rotation Offset" ""
+			(at 99.06 106.68 0)
+			(effects
+				(font
+					(size 1.27 1.27)
+				)
+				(hide yes)
+			)
+		)
 		(pin "2"
 		)
@@
 			)
 		)
+		(property "JLCPCB Rotation Offset" ""
+			(at 127 48.26 0)
+			(effects
+				(font
+					(size 1.27 1.27)
+				)
+				(hide yes)
+			)
+		)
 		(pin "2"
 		)
@@
 			)
 		)
+		(property "JLCPCB Rotation Offset" ""
+			(at 25.4 175.26 0)
+			(effects
+				(font
+					(size 1.27 1.27)
+				)
+				(hide yes)
+			)
+		)
 		(pin "2"
 		)
@@
 			)
 		)
-		(property "LCSC Part #" "C1521934"
+		(property "LCSC Part #" "C1521935"
+			(at 208.28 99.06 0)
+			(effects
+				(font
+					(size 1.27 1.27)
+				)
+				(hide yes)
+			)
+		)
+		(property "JLCPCB Rotation Offset" ""
 			(at 208.28 99.06 0)
 			(effects
@@
 		(unit 1)
 		(exclude_from_sim no)
-		(in_bom yes)
+		(in_bom no)
 		(on_board yes)
 		(dnp no)
@@
 			)
 		)
-		(property "LCSC Part #" "C2913924"
+		(property "LCSC Part #" ""
+			(at 73.66 71.12 0)
+			(effects
+				(font
+					(size 1.27 1.27)
+				)
+				(hide yes)
+			)
+		)
+		(property "JLCPCB Rotation Offset" ""
 			(at 73.66 71.12 0)
 			(effects
@@
 			)
 		)
+		(property "JLCPCB Rotation Offset" "270"
+			(at 58.42 152.4 0)
+			(effects
+				(font
+					(size 1.27 1.27)
+				)
+				(hide yes)
+			)
+		)
 		(pin "1"
 		)
@@
 		(on_board yes)
 		(dnp no)
-		(property "Reference" "#GND24"
+		(property "Reference" "#GND024"
 			(at 25.4 185.42 0)
 			(effects
@@
 			(project ""
 				(path "/e6275eb3-d183-4a15-8a8c-dffc95cf456c/7ef72fdc-db96-4316-aacb-30b112fc5f48"
-					(reference "#GND24")
+					(reference "#GND024")
 					(unit 1)
 				)
@@
 			)
 		)
+		(property "JLCPCB Rotation Offset" ""
+			(at 99.06 104.14 0)
+			(effects
+				(font
+					(size 1.27 1.27)
+				)
+				(hide yes)
+			)
+		)
 		(pin "1"
 		)
@@
 			)
 		)
-		(property "LCSC Part #" "C1179056"
+		(property "LCSC Part #" "C7431354"
+			(at 55.88 177.8 0)
+			(effects
+				(font
+					(size 1.27 1.27)
+				)
+				(hide yes)
+			)
+		)
+		(property "JLCPCB Rotation Offset" ""
 			(at 55.88 177.8 0)
 			(effects
@@
 			)
 		)
+		(property "JLCPCB Rotation Offset" ""
+			(at 127 101.6 0)
+			(effects
+				(font
+					(size 1.27 1.27)
+				)
+				(hide yes)
+			)
+		)
 		(pin "1"
 		)
@@
 		(on_board yes)
 		(dnp no)
-		(property "Reference" "#GND29"
+		(property "Reference" "#GND029"
 			(at 127 60.96 0)
 			(effects
@@
 			(project ""
 				(path "/e6275eb3-d183-4a15-8a8c-dffc95cf456c/7ef72fdc-db96-4316-aacb-30b112fc5f48"
-					(reference "#GND29")
+					(reference "#GND029")
 					(unit 1)
 				)
@@
 			(at 96.52 119.38 0)
 			(effects
+				(font
+					(size 1.27 1.27)
+				)
+				(hide yes)
+			)
+		)
+		(property "JLCPCB Rotation Offset" ""
+			(at 96.52 119.38 0)
+			(effects

Commit message: Final adjustements to production files for JLC
Connections:
- no-connect marks 0 -> 27
Changed lines of the file:
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@@
 		(color 0 0 0 0)
 	)
+	(no_connect
+		(at 256.54 142.24)
+	)
+	(no_connect
+		(at 213.36 55.88)
+	)
+	(no_connect
+		(at 215.9 157.48)
+	)
+	(no_connect
+		(at 147.32 157.48)
+	)
+	(no_connect
+		(at 220.98 157.48)
+	)
+	(no_connect
+		(at 256.54 139.7)
+	)
+	(no_connect
+		(at 218.44 55.88)
+	)
+	(no_connect
+		(at 233.68 157.48)
+	)
+	(no_connect
+		(at 256.54 66.04)
+	)
+	(no_connect
+		(at 231.14 55.88)
+	)
+	(no_connect
+		(at 208.28 157.48)
+	)
+	(no_connect
+		(at 228.6 157.48)
+	)
+	(no_connect
+		(at 134.62 93.98)
+	)
+	(no_connect
+		(at 256.54 137.16)
+	)
+	(no_connect
+		(at 226.06 157.48)
+	)
+	(no_connect
+		(at 195.58 157.48)
+	)
+	(no_connect
+		(at 134.62 68.58)
+	)
+	(no_connect
+		(at 223.52 157.48)
+	)
+	(no_connect
+		(at 152.4 157.48)
+	)
+	(no_connect
+		(at 134.62 99.06)
+	)
+	(no_connect
+		(at 190.5 157.48)
+	)
+	(no_connect
+		(at 215.9 55.88)
+	)
+	(no_connect
+		(at 238.76 55.88)
+	)
+	(no_connect
+		(at 256.54 134.62)
+	)
+	(no_connect
+		(at 228.6 55.88)
+	)
+	(no_connect
+		(at 236.22 55.88)
+	)
+	(no_connect
+		(at 205.74 157.48)
+	)
 	(bus_entry
 		(at 198.12 27.94)
@@
 	(global_label "AUD1"
 		(shape bidirectional)
-		(at 228.6 27.94 0)
+		(at 228.6 27.94 270)
 		(fields_autoplaced yes)
 		(effects
@@
 				(size 1.016 1.016)
 			)
-			(justify left)
+			(justify right top)
 		)
 		(property "Intersheetrefs" "${INTERSHEET_REFS}"
-			(at 235.7958 27.94 0)
+			(at 228.6 35.1358 90)
 			(effects
 				(font
 					(size 1.27 1.27)
 				)
-				(justify left)
+				(justify right)
 				(hide yes)
 			)
@@
 	(global_label "3V3"
 		(shape bidirectional)
-		(at 71.12 182.88 0)
+		(at 73.66 182.88 0)
 		(fields_autoplaced yes)
 		(effects
@@
 		)
 		(property "Intersheetrefs" "${INTERSHEET_REFS}"
-			(at 78.5716 182.88 0)
+			(at 81.1116 182.88 0)
 			(effects
 				(font
@@
 	(global_label "3V3"
 		(shape bidirectional)
-		(at 17.78 172.72 0)
+		(at 17.78 172.72 180)
 		(fields_autoplaced yes)
 		(effects
@@
 				(size 1.2446 1.2446)
 			)
-			(justify left)
+			(justify right)
 		)
 		(property "Intersheetrefs" "${INTERSHEET_REFS}"

Commit message: Update BOM from 0402 to 0603 where relevant
Parts:
- C10: LCSC Part # C15195 -> C43253
- R1, R2, R4, R5: LCSC Part # C25744 -> C103199
- R3: LCSC Part # C11702 -> C107079
Changed lines of the file:
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@@
 			)
 		)
-		(property "LCSC Part #" "C25744"
+		(property "LCSC Part #" "C103199"
 			(at 127 109.22 0)
 			(effects
@@
 			)
 		)
-		(property "LCSC Part #" "C25744"
+		(property "LCSC Part #" "C103199"
 			(at 99.06 106.68 0)
 			(effects
@@
 			)
 		)
-		(property "LCSC Part #" "C11702"
+		(property "LCSC Part #" "C107079"
 			(at 127 48.26 0)
 			(effects
@@
 			)
 		)
-		(property "LCSC Part #" " C15195"
+		(property "LCSC Part #" "C43253"
 			(at 25.4 175.26 0)
 			(effects
@@
 			)
 		)
-		(property "LCSC Part #" "C25744"
+		(property "LCSC Part #" "C103199"
 			(at 99.06 104.14 0)
 			(effects
@@
 			)
 		)
-		(property "LCSC Part #" "C25744"
+		(property "LCSC Part #" "C103199"
 			(at 127 101.6 0)
 			(effects
