File: PokeyMax4s/Audio_filter.kicad_sch (KiCad schematic)
At the start: 16 parts, among them U1 TSV854IQ4T

Commit message: PokeyMax 4s fabrication files
Parts:
- AUD0: now left out of the parts list
Changed lines of the file:
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@@
 		(unit 1)
 		(exclude_from_sim no)
-		(in_bom yes)
+		(in_bom no)
 		(on_board yes)
 		(dnp no)

Commit message: Add A4 to PokeyMax 4s
Reroute accordingly
Connections:
- net AUDF3 renamed RIGHT
- net AUDF4 renamed LEFT
- net LVLA21 renamed DIGITAL_AUDIO_OUT
Changed lines of the file:
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@@
 		)
 	)
-	(label "AUDF4"
+	(label "LEFT"
 		(at 219.71 101.6 0)
 		(fields_autoplaced yes)
@@
 		)
 	)
-	(label "AUDF3"
+	(label "RIGHT"
 		(at 219.71 104.14 0)
 		(fields_autoplaced yes)
@@
 		)
 	)
-	(global_label "LVLA21"
+	(global_label "DIGITAL_AUDIO_OUT"
 		(shape bidirectional)
 		(at 226.06 106.68 270)
