File: PokeyMax4s/PokeyMax4s.kicad_pcb (KiCad board)
At the start: 2 copper layers, 20.2 x 52.8 mm, 49 parts, among them J1 GTIA 15, J2 A4, U1 TSV854IQ4T, U2 74CB3T16210, U3 MAX10, U4 74CB3T16210, X1 50MHz

Commit message: Fix typo on 4s board
Other:
- board text added: "GTIA 15"
Changed lines of the file:
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@@
 		)
 	)
-	(gr_text "GTIO 15"
+	(gr_text "GTIA 15"
 		(at 154.206 93.425 -90)
 		(layer "B.SilkS")
@@
 			(justify right mirror)
 		)
-		(render_cache "GTIO 15" 270
+		(render_cache "GTIA 15" 270
 			(polygon
 				(pts
-					(xy 154.055521 96.743576) (xy 154.375186 96.743576) (xy 154.375186 96.917086) (xy 154.0352 96.917086)
-					(xy 154.041864 96.965215) (xy 154.057774 97.009764) (xy 154.081863 97.049788) (xy 154.113064 97.084343)
-					(xy 154.150311 97.112488) (xy 154.192535 97.133277) (xy 154.23867 97.145769) (xy 154.287649 97.149019)
-					(xy 154.336665 97.142169) (xy 154.381411 97.125761) (xy 154.421206 97.100954) (xy 154.455371 97.068907)
-					(xy 154.483225 97.030779) (xy 154.504088 96.987727) (xy 154.517281 96.940911) (xy 154.522122 96.891489)
-					(xy 154.523295 96.820756) (xy 154.68684 96.820756) (xy 154.68684 96.89696) (xy 154.68427 96.94164)
-					(xy 154.67716 96.985159) (xy 154.665751 97.027253) (xy 154.650286 97.067658) (xy 154.631004 97.106112)
-					(xy 154.608148 97.14235) (xy 154.581959 97.176108) (xy 154.552677 97.207124) (xy 154.520545 97.235133)
-					(xy 154.485803 97.259873) (xy 154.448693 97.281078) (xy 154.409456 97.298486) (xy 154.368334 97.311834)
-					(xy 154.325567 97.320856) (xy 154.281397 97.325291) (xy 154.236065 97.324874) (xy 154.189268 97.318157)
-					(xy 154.143842 97.304747) (xy 154.100233 97.285299) (xy 154.058888 97.26047) (xy 154.020253 97.230916)
-					(xy 153.984775 97.197293) (xy 153.952898 97.160258) (xy 153.925071 97.120467) (xy 153.901738 97.078576)
-					(xy 153.883346 97.035242) (xy 153.870341 96.99112) (xy 153.86317 96.946868) (xy 153.862279 96.903141)
-					(xy 153.868114 96.860597) (xy 153.88112 96.81989) (xy 153.901745 96.781678) (xy 153.932306 96.757212)
-					(xy 153.970824 96.74709) (xy 154.015296 96.743843)
+					(xy 154.055521 96.590387) (xy 154.375186 96.590387) (xy 154.375186 96.763897) (xy 154.0352 96.763897)
+					(xy 154.041864 96.812026) (xy 154.057774 96.856575) (xy 154.081863 96.896599) (xy 154.113064 96.931154)
+					(xy 154.150311 96.959299) (xy 154.192535 96.980088) (xy 154.23867 96.99258) (xy 154.287649 96.99583)
+					(xy 154.336665 96.98898) (xy 154.381411 96.972572) (xy 154.421206 96.947765) (xy 154.455371 96.915718)
+					(xy 154.483225 96.87759) (xy 154.504088 96.834538) (xy 154.517281 96.787722) (xy 154.522122 96.7383)
+					(xy 154.523295 96.667567) (xy 154.68684 96.667567) (xy 154.68684 96.743771) (xy 154.68427 96.788451)
+					(xy 154.67716 96.83197) (xy 154.665751 96.874064) (xy 154.650286 96.914469) (xy 154.631004 96.952923)
+					(xy 154.608148 96.989161) (xy 154.581959 97.022919) (xy 154.552677 97.053935) (xy 154.520545 97.081944)
+					(xy 154.485803 97.106684) (xy 154.448693 97.127889) (xy 154.409456 97.145297) (xy 154.368334 97.158645)
+					(xy 154.325567 97.167667) (xy 154.281397 97.172102) (xy 154.236065 97.171685) (xy 154.189268 97.164968)
+					(xy 154.143842 97.151558) (xy 154.100233 97.13211) (xy 154.058888 97.107281) (xy 154.020253 97.077727)
+					(xy 153.984775 97.044104) (xy 153.952898 97.007069) (xy 153.925071 96.967278) (xy 153.901738 96.925387)
+					(xy 153.883346 96.882053) (xy 153.870341 96.837931) (xy 153.86317 96.793679) (xy 153.862279 96.749952)
+					(xy 153.868114 96.707408) (xy 153.88112 96.666701) (xy 153.901745 96.628489) (xy 153.932306 96.604023)
+					(xy 153.970824 96.593901) (xy 154.015296 96.590654)
 				)
 			)
 			(polygon
 				(pts
-					(xy 154.525249 96.145865) (xy 154.691138 96.145865) (xy 154.691138 96.626535) (xy 154.526421 96.626535)
-					(xy 154.526421 96.472955) (xy 153.874 96.472955) (xy 153.874 96.29495) (xy 154.525249 96.29495)
+					(xy 154.525249 95.992676) (xy 154.691138 95.992676) (xy 154.691138 96.473346) (xy 154.526421 96.473346)
+					(xy 154.526421 96.319766) (xy 153.874 96.319766) (xy 153.874 96.141761) (xy 154.525249 96.141761)
 				)
 			)
 			(polygon
 				(pts
-					(xy 153.874 95.820142) (xy 154.68938 95.820142) (xy 154.68938 95.995997) (xy 153.874 95.995997)
+					(xy 153.874 95.666953) (xy 154.68938 95.666953) (xy 154.68938 95.842808) (xy 153.874 95.842808)
 				)
 			)
 			(polygon
 				(pts
-					(xy 154.31852 94.853718) (xy 154.359553 94.860014) (xy 154.3992 94.870253) (xy 154.437248 94.884225)
-					(xy 154.473482 94.901723) (xy 154.507689 94.922537) (xy 154.539654 94.946458) (xy 154.569163 94.973279)
-					(xy 154.596003 95.00279) (xy 154.619958 95.034784) (xy 154.640816 95.06905) (xy 154.658361 95.105381)
-					(xy 154.67238 95.143568) (xy 154.682659 95.183402) (xy 154.688983 95.224674) (xy 154.691138 95.267177)
-					(xy 154.688983 95.309679) (xy 154.682659 95.350951) (xy 154.67238 95.390785) (xy 154.658361 95.428972)
-					(xy 154.640816 95.465303) (xy 154.619958 95.499569) (xy 154.596003 95.531563) (xy 154.569163 95.561074)
-					(xy 154.539654 95.587895) (xy 154.507689 95.611817) (xy 154.473482 95.63263) (xy 154.437248 95.650128)
-					(xy 154.3992 95.6641) (xy 154.359553 95.674339) (xy 154.31852 95.680635) (xy 154.276316 95.68278)
-					(xy 154.233919 95.680635) (xy 154.192743 95.674339) (xy 154.152997 95.6641) (xy 154.11489 95.650128)
-					(xy 154.078631 95.63263) (xy 154.044428 95.611817) (xy 154.012492 95.587895) (xy 153.98303 95.561074)
-					(xy 153.956251 95.531563) (xy 153.932365 95.499569) (xy 153.911581 95.465303) (xy 153.894107 95.428972)
-					(xy 153.880152 95.390785) (xy 153.869926 95.350951) (xy 153.863637 95.309679) (xy 153.861494 95.267177)
-					(xy 154.029338 95.267177) (xy 154.034356 95.317084) (xy 154.048749 95.363561) (xy 154.071523 95.405614)
-					(xy 154.101683 95.44225) (xy 154.138236 95.472474) (xy 154.180188 95.495293) (xy 154.226546 95.509713)
-					(xy 154.276316 95.514741) (xy 154.326022 95.509713) (xy 154.372331 95.495293) (xy 154.414249 95.472474)
-					(xy 154.450779 95.44225) (xy 154.480925 95.405614) (xy 154.503691 95.363561) (xy 154.518081 95.317084)
-					(xy 154.523099 95.267177) (xy 154.518081 95.217325) (xy 154.503691 95.170875) (xy 154.480925 95.128825)
-					(xy 154.450779 95.092177) (xy 154.414249 95.06193) (xy 154.372331 95.039087) (xy 154.326022 95.024648)
-					(xy 154.276316 95.019612) (xy 154.226546 95.024648) (xy 154.180188 95.039087) (xy 154.138236 95.06193)
-					(xy 154.101683 95.092177) (xy 154.071523 95.128825) (xy 154.048749 95.170875) (xy 154.034356 95.217325)
-					(xy 154.029338 95.267177) (xy 153.861494 95.267177) (xy 153.863637 95.224674) (xy 153.869926 95.183402)
-					(xy 153.880152 95.143568) (xy 153.894107 95.105381) (xy 153.911581 95.06905) (xy 153.932365 95.034784)
-					(xy 153.956251 95.00279) (xy 153.98303 94.973279) (xy 154.012492 94.946458) (xy 154.044428 94.922537)
-					(xy 154.078631 94.901723) (xy 154.11489 94.884225) (xy 154.152997 94.870253) (xy 154.192743 94.860014)
-					(xy 154.233919 94.853718) (xy 154.276316 94.851573)
+					(xy 154.612981 95.06807) (xy 154.649216 95.084037) (xy 154.682192 95.111715) (xy 154.703889 95.14817)
+					(xy 154.711925 95.192064) (xy 154.71185 95.198007) (xy 154.70343 95.240875) (xy 154.682736 95.276433)
+					(xy 154.651345 95.303602) (xy 154.610831 95.321301) (xy 153.874 95.534085) (xy 153.874 95.341426)
+					(xy 154.032073 95.304497) (xy 154.032073 95.259556) (xy 154.201285 95.259556) (xy 154.43693 95.192341)
+					(xy 154.201285 95.12747) (xy 154.201285 95.259556) (xy 154.032073 95.259556) (xy 154.032073 95.086046)
+					(xy 153.874 95.042278) (xy 153.874 94.848642)
 				)
 			)
@@
 					(xy 153.874 94.147763) (xy 154.529743 94.147763) (xy 154.568845 94.148958) (xy 154.607553 94.156255)
 					(xy 154.642861 94.174918) (xy 154.653036 94.18352) (xy 154.678307 94.21365) (xy 154.693373 94.249974)
-					(xy 154.697782 94.292354) (xy 154.697782 94.424441) (xy 154.525249 94.424441) (xy 154.525249 94.317951)
+					(xy 154.697782 94.292355) (xy 154.697782 94.424441) (xy 154.525249 94.424441) (xy 154.525249 94.317951)
 					(xy 153.874 94.317951)
 				)
@@
 					(xy 154.388836 93.638724) (xy 154.402535 93.676746) (xy 154.410215 93.717098) (xy 154.411725 93.745055)
 					(xy 154.411725 93.842557) (xy 154.523099 93.842557) (xy 154.523099 93.532271) (xy 154.691138 93.532271)
-					(xy 154.691138 94.004929) (xy 154.376944 94.004929) (xy 154.336264 94.000983) (xy 154.298744 93.984749)
+					(xy 154.691138 94.00493) (xy 154.376944 94.00493) (xy 154.336264 94.000983) (xy 154.298744 93.984749)
 					(xy 154.280615 93.969172) (xy 154.258327 93.936977) (xy 154.248786 93.898806) (xy 154.24818 93.882808)
 					(xy 154.24818 93.761859) (xy 154.242232 93.722037) (xy 154.22219 93.682564) (xy 154.190179 93.654043)
 					(xy 154.148453 93.641182) (xy 154.142667 93.64091) (xy 154.099802 93.64843) (xy 154.063825 93.670292)
 					(xy 154.038692 93.703256) (xy 154.028361 93.744078) (xy 154.036467 93.787666) (xy 154.06126 93.823286)
-					(xy 154.098181 93.846706) (xy 154.136848 93.853864) (xy 154.142667 93.853694) (xy 154.142667 94.026227)
-					(xy 154.099942 94.023271) (xy 154.059153 94.014075) (xy 154.0208 93.999139) (xy 153.985386 93.978963)
-					(xy 153.953414 93.954046) (xy 153.925386 93.924886) (xy 153.901804 93.891985) (xy 153.883171 93.855841)
+					(xy 154.098181 93.846706) (xy 154.136848 93.853864) (xy 154.142667 93.853694) (xy 154.142667 94.026228)
+					(xy 154.099942 94.023271) (xy 154.059153 94.014075) (xy 154.0208 93.99914) (xy 153.985386 93.978963)
+					(xy 153.953414 93.954046) (xy 153.925386 93.924887) (xy 153.901804 93.891985) (xy 153.883171 93.855841)
 					(xy 153.869988 93.816953) (xy 153.862759 93.775821) (xy 153.861494 93.7474) (xy 153.864773 93.706913)
-					(xy 153.87377 93.668284) (xy 153.893914 93.620425) (xy 153.922429 93.577681) (xy 153.95829 93.541088)
-					(xy 154.000471 93.51168) (xy 154.047945 93.490492) (xy 154.086409 93.480619)
+					(xy 153.87377 93.668284) (xy 153.893914 93.620425) (xy 153.922429 93.577682) (xy 153.95829 93.541088)
+					(xy 154.000471 93.51168) (xy 154.047945 93.490493) (xy 154.086409 93.480619)
 				)
 			)

Commit message: Bump rev number to 1.1
Connections:
- U2 pad 45: AUD1 -> LIN22
- U3 pad C12: AUD1 -> LIN22
Routing:
- net LIN22: track 0.00 -> 26.6 mm, vias 0 -> 2
- net AUD1: track 65.9 -> 39.9 mm, vias 6 -> 4
Other:
- board text added: "Rev 1.1 Original design by Foft in 2024 https://forums.atariage.com/profile/8458-foft/ Redrawn by ScreamingAtTheRadio in 2024 https://github.com/bleroy/pokeymax/tree/main/PokeyMax4s"
- board text removed: "Original design by Foft in 2024 https://forums.atariage.com/profile/8458-foft/ Redrawn by ScreamingAtTheRadio in 2024 https://github.com/bleroy/pokeymax/tree/main/PokeyMax4s"
